Commit message: Add laser link

File: src/pipibot_description/urdf/pipibot.urdf (robot description, URDF)
Before this commit: robot pipi_bot, 1 links, 0 joints
Links:
- added link laser; visual mesh filename=package://pipibot_description/meshes/laser.stl scale=0.001 0.001 0.001
Joints:
- added joint base_to_laser: type fixed, parent base_link, child laser, origin xyz=0.0 0.0 0.1 rpy=0 0 0

Commit message: With test codes

File: src/pipibot_description/urdf/pipibot.urdf (robot description, URDF)
Before this commit: robot pipi_bot, 2 links, 1 joints
Joints:
- joint base_to_laser: origin xyz=0.0 0.0 0.1 rpy=0 0 0 -> xyz=0.0 0.0 0.08 rpy=0 0 0
